File: VFD display 1.kicad_pcb (KiCad board)
At the start: 2 copper layers, 100 x 50 mm, 166 parts, among them J1 Conn_01x08_Pin, J2 Conn_01x08_Socket, Q1 BC846, Q10 BC846, Q11 BC856, Q12 BC846, Q13 BC856, Q14 BC846, Q15 BC856, Q16 BC846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

Commit message: silkscreen and production files
Other:
- board text added: "32bit long shift register"
- board text added: "filament voltage"
- board text removed: "74HC595"
